Commit message: Sync

File: sawyer_description_openrave/urdf/real_sawyer_arm_only.urdf (robot description, URDF)
Before this commit: robot sawyer, 12 links, 11 joints
Links:
- removed link right_gripper
- removed link right_gripper_base
- added link head, mass 1.5795; collision sphere radius=0.18; visual mesh filename=package://sawyer_description_openrave/meshes/sawyer_pv/head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
- added link head_camera
- added link right_arm_itb, mass 0.0001
- added link right_hand_camera
- added link right_l1_2, mass 1.0E-08; collision cylinder length=0.14 radius=0.07
- added link right_l2_2, mass 1.0E-08; collision sphere radius=0.06
- added link right_l4_2, mass 1.0E-08; collision sphere radius=0.06
- added link right_torso_itb, mass 0.0001
- added link right_wrist
- added link screen, mass 0.0001; collision sphere radius=0.001; visual box size=0.24 0.14 0.002
- link right_arm_base_link: geometry collision cylinder length=0.24 radius=0.08; visual mesh filename=package://sawyer_description_openrave/meshes/sawyer_pv/base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
- link right_l0: geometry collision sphere radius=0.07; visual mesh filename=package://sawyer_description_openrave/meshes/sawyer_mp3/l0.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
- link right_l1: geometry collision sphere radius=0.07; visual mesh filename=package://sawyer_description_openrave/meshes/sawyer_mp3/l1.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
- link right_l2: geometry collision cylinder length=0.34 radius=0.06; visual mesh filename=package://sawyer_description_openrave/meshes/sawyer_pv/l2.D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
- link right_l3: geometry collision sphere radius=0.06; visual mesh filename=package://sawyer_description_openrave/meshes/sawyer_pv/l3.D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
- link right_l4: geometry collision cylinder length=0.30 radius=0.045; visual mesh filename=package://sawyer_description_openrave/meshes/sawyer_pv/l4.D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
- link right_l5: geometry collision sphere radius=0.06; visual mesh filename=package://sawyer_description_openrave/meshes/sawyer_pv/l5.D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
- link right_l6: geometry collision cylinder length=0.05 radius=0.055; visual mesh filename=package://sawyer_description_openrave/meshes/sawyer_mp1/l6.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
Joints:
- removed joint right_gripper_base
- removed joint right_gripper_endpoint
- added joint display_joint: type fixed, parent head, child screen, origin xyz=0.03 0.0 0.105 rpy=1.57079632679 0 1.57079632679
- added joint head_camera: type fixed, parent head, child head_camera, origin xyz=0.0253976919969 -0.000870932656271 0.215696810568 rpy=-2.12362578457 0.00914483957425 -1.57079632679, axis 0 0 0
- added joint head_pan: type revolute, parent right_l0, child head, origin xyz=-0.00043503123114 0.000635456478455 0.2965 rpy=-0.000375610612151 -0.000717773645631 0.060618282317, axis 0 0 1, limit lower=-5.0952 upper=0.9064 effort=8 velocity=1.8
- added joint right_arm_itb: type fixed, parent right_l4, child right_arm_itb, origin xyz=-.055 0 .075 rpy=0 -1.57079632679 0, axis 0 0 1
- added joint right_hand_camera: type fixed, parent right_l5, child right_hand_camera, origin xyz=0.0382275754565 -0.032511331905 0.0686165502955 rpy=-0.445734774695 1.55629550314 -0.429789630424, axis 0 0 0
- added joint right_j1_2: type fixed, parent right_l1, child right_l1_2, origin xyz=0 0 0 rpy=0 0 0, axis 0 0 1
- added joint right_j2_2: type fixed, parent right_l2, child right_l2_2, origin xyz=0 0 0 rpy=0 0 0, axis 0 0 1
- added joint right_j4_2: type fixed, parent right_l4, child right_l4_2, origin xyz=0 0 0 rpy=0 0 0, axis 0 0 1
- added joint right_torso_itb: type fixed, parent right_l0, child right_torso_itb, origin xyz=-.055 0 .22 rpy=0 -1.57079632679 0, axis 0 0 1
- added joint right_wrist: type fixed, parent right_l5, child right_wrist, origin xyz=0 0 0.10541 rpy=1.57079632679 0 0, axis 0 0 0

Commit message: More tests with OpenRAVE and Sawyer

File: sawyer_description_openrave/urdf/real_sawyer_arm_only.urdf (robot description, URDF)
Before this commit: robot sawyer, 20 links, 19 joints
Links:
- link head: geometry collision cylinder length=0.28 radius=0.065; visual mesh filename=package://sawyer_description_openrave/meshes/sawyer_pv/head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
- link right_arm_base_link: geometry collision cylinder length=0.24 radius=0.11; visual mesh filename=package://sawyer_description_openrave/meshes/sawyer_pv/base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
- link right_l2: mass 1.745 -> 1.7251
- link screen: geometry collision box size=0.32 0.22 0.1; visual box size=0.24 0.14 0.002
Joints:
- joint display_joint: origin xyz=0.03 0.0 0.105 rpy=1.57079632679 0 1.57079632679 -> xyz=0.03 0.0 0.105 rpy=1.5708 0 1.5708
- joint head_camera: origin xyz=0.0253976919969 -0.000870932656271 0.215696810568 rpy=-2.12362578457 0.00914483957425 -1.57079632679 -> xyz=0.0228027 0 0.216572 rpy=-2.1293 0 -1.5708
- joint head_pan: origin xyz=-0.00043503123114 0.000635456478455 0.2965 rpy=-0.000375610612151 -0.000717773645631 0.060618282317 -> xyz=0 0 0.2965 rpy=0 0 0
- joint right_arm_itb: origin xyz=-.055 0 .075 rpy=0 -1.57079632679 0 -> xyz=-.055 0 .075 rpy=0 -1.5708 0
- joint right_hand: origin xyz=0 0 0.0245 rpy=0 0 1.570796 -> xyz=0 0 0.0245 rpy=0 0 1.5708
- joint right_hand_camera: origin xyz=0.0382275754565 -0.032511331905 0.0686165502955 rpy=-0.445734774695 1.55629550314 -0.429789630424 -> xyz=0.039552 -0.033 0.0695 rpy=0 1.5708 0
- joint right_j0: origin xyz=0.000163597 5.46084e-05 0.0795794219 rpy=-0.0002985644 0.0018972651 4.67207e-05 -> xyz=0 0 0.08 rpy=0 0 0
- joint right_j1: origin xyz=0.0807732027 0.0500167937 0.237 rpy=-1.57005949279 1.56949847329 -0.0008032605 -> xyz=0.081 0.05 0.237 rpy=-1.5708 1.5708 0
- joint right_j2: origin xyz=-0.0011561 -0.1402394172 0.1425177448 rpy=1.56982185629 -0.0008951969 0.0024593204 -> xyz=0 -0.14 0.1425 rpy=1.5708 0 0
- joint right_j3: origin xyz=-0.0003042945 -0.0421041777 0.2600595397 rpy=-1.57152985219 -0.0004637381 0.00025132 -> xyz=0 -0.042 0.26 rpy=-1.5708 0 0
- joint right_j4: origin xyz=-4.14656e-05 -0.1247526357 -0.1266411523 rpy=1.57148053569 -0.0006765717 -0.0004526017 -> xyz=0 -0.125 -0.1265 rpy=1.5708 0 0
- joint right_j5: origin xyz=-0.0001236812 0.0307252196 0.2746521054 rpy=-1.56869259669 0.0005321883 0.0007813353 -> xyz=0 0.031 0.275 rpy=-1.5708 0 0
- joint right_j6: origin xyz=0.0001362646 -0.1098066995 0.1050523612 rpy=-1.56987330589 -0.1773123624 3.1421484795 -> xyz=0 -0.11 0.1053 rpy=-1.5708 -0.17453 3.1416
- joint right_torso_itb: origin xyz=-.055 0 .22 rpy=0 -1.57079632679 0 -> xyz=-.055 0 .22 rpy=0 -1.5708 0
- joint right_wrist: origin xyz=0 0 0.10541 rpy=1.57079632679 0 0 -> xyz=0 0 0.10541 rpy=1.5708 0 0
